File: PCB/MirZ21_Sub-D_Renamed_U.brd (EAGLE design)
At the start: 65.2 x 45.6 mm, 32 parts, among them CON1 M04B4B-ZR4P, CON3 M04, IC1 7805, J1 SOLDERJUMPERTRACE, T1 CON-HARTING-ML_ML4ML4_FEMALE

Commit message: Added ToDos for next revision
Parts:
- added D2: PESD1CAN, diode:SOT23
Connections:
- net CAN_H: now also D2.1
- net CAN_L: now also D2.2
- net GND: now also D2.3
Changed lines of the file:
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@@
 <attribute name="VALUE" x="56.515" y="13.6525" size="1.27" layer="27" rot="R90"/>
+</element>
+<element name="D2" library="diode" library_urn="urn:adsk.eagle:library:210" package="SOT23" package3d_urn="urn:adsk.eagle:package:43389/2" value="PESD1CAN" x="-11" y="-19" smashed="yes">
+<attribute name="NAME" x="-12.905" y="-17.095" size="1.27" layer="25"/>
+<attribute name="POPULARITY" value="0" x="-11" y="-19" size="1.778" layer="27" display="off"/>
+<attribute name="VALUE" x="-12.905" y="-22.175" size="1.27" layer="27"/>
 </element>
 </elements>
@@
 <wire x1="52.07" y1="14.28868125" x2="52.07" y2="7.62" width="0.508" layer="1"/>
 <wire x1="51.9938" y1="18.02011875" x2="51.9938" y2="14.36488125" width="0.508" layer="1"/>
+<contactref element="D2" pad="3"/>
+<wire x1="20.7645" y1="1.905" x2="-11" y2="-17.9" width="0" layer="19" extent="1-1"/>
 </signal>
 <signal name="+5V">
@@
 <wire x1="47.3202" y1="15.8496" x2="45.3898" y2="17.78" width="0.254" layer="1"/>
 <wire x1="48.26" y1="15.09513125" x2="47.50553125" y2="15.8496" width="0.254" layer="1"/>
+<contactref element="D2" pad="1"/>
+<wire x1="-11.95" y1="-20.1" x2="41.275" y2="1.905" width="0" layer="19" extent="1-1"/>
 </signal>
 <signal name="CAN_L">
@@
 <wire x1="48.2346" y1="20.9804" x2="50.8254" y2="20.9804" width="0.254" layer="16"/>
 <wire x1="50.8254" y1="20.9804" x2="51.9712" y2="22.1262" width="0.254" layer="16"/>
+<contactref element="D2" pad="2"/>
+<wire x1="-10.05" y1="-20.1" x2="43.815" y2="1.905" width="0" layer="19" extent="1-1"/>
 </signal>
 <signal name="SPK+">
