File: PCB/MirZ21_Sub-D_Renamed_U.sch (EAGLE design)
At the start: 32 parts, among them CON1 M04B4B-ZR4P, CON3 M04, IC1 7805, J1 SOLDERJUMPERTRACE, T1 CON-HARTING-ML_ML4ML4_FEMALE

Commit message: Added ToDos for next revision
Parts:
- added D2: PESD1CAN, diode:PESD1CAN
Connections:
- net CAN_H: now also D2.1
- net CAN_L: now also D2.2
- net GND: now also D2.3
Other:
- note added: "ToDo: - Pinbelegung Märklin Kabel korrigieren - ESP32 ein bisschen nach rechts verschieben weil es Versionen gibt welche nicht in das Gehäuse passen - PESD2CAN platzieren"
Changed lines of the file:
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@@
 <part name="J1" library="SparkFun-Retired" deviceset="SOLDERJUMPER" device="TRACE" value="SOLDERJUMPERTRACE"/>
 <part name="JP1" library="SparkFun-Connectors" deviceset="M02" device="PTH" value="Test"/>
+<part name="D2" library="diode" library_urn="urn:adsk.eagle:library:210" deviceset="PESD1CAN" device="" package3d_urn="urn:adsk.eagle:package:43389/2"/>
+<part name="GND21" library="supply1" library_urn="urn:adsk.eagle:library:371" deviceset="GND" device=""/>
 </parts>
 <sheets>
@@
   (Old 0.7mm)
 </text>
+<text x="40.64" y="15.24" size="1.778" layer="94">ToDo:
+- Pinbelegung Märklin Kabel korrigieren
+- ESP32 ein bisschen nach rechts verschieben
+  weil es Versionen gibt welche nicht in das
+  Gehäuse passen
+- PESD2CAN platzieren</text>
 </plain>
 <instances>
@@
 <attribute name="VALUE" x="114.3" y="167.64" size="1.778" layer="96" rot="MR90"/>
 <attribute name="NAME" x="125.222" y="170.18" size="1.778" layer="95" rot="MR90"/>
+</instance>
+<instance part="D2" gate="G$1" x="58.42" y="172.72" smashed="yes" rot="R270">
+<attribute name="NAME" x="63.5" y="177.8" size="1.778" layer="95" rot="R270"/>
+<attribute name="VALUE" x="50.8" y="177.8" size="1.778" layer="96" rot="R270"/>
+</instance>
+<instance part="GND21" gate="1" x="58.42" y="165.1" smashed="yes">
+<attribute name="VALUE" x="54.61" y="162.56" size="1.778" layer="96"/>
 </instance>
 </instances>
@@
 <pinref part="T1" gate="1" pin="1"/>
 <pinref part="GND20" gate="1" pin="GND"/>
+</segment>
+<segment>
+<pinref part="D2" gate="G$1" pin="3"/>
+<pinref part="GND21" gate="1" pin="GND"/>
 </segment>
 </net>
@@
 <label x="30.48" y="193.04" size="1.778" layer="95"/>
 <pinref part="CON3" gate="G$1" pin="1"/>
-<wire x1="73.66" y1="193.04" x2="25.4" y2="193.04" width="0.1524" layer="91"/>
+<wire x1="73.66" y1="193.04" x2="60.96" y2="193.04" width="0.1524" layer="91"/>
+<wire x1="60.96" y1="193.04" x2="25.4" y2="193.04" width="0.1524" layer="91"/>
 <wire x1="25.4" y1="187.96" x2="25.4" y2="193.04" width="0.1524" layer="91"/>
 <pinref part="CON1" gate="G$1" pin="1"/>
@@
 <label x="73.66" y="205.74" size="1.778" layer="95" rot="R90"/>
 <label x="30.48" y="218.44" size="1.778" layer="95"/>
+<pinref part="D2" gate="G$1" pin="1"/>
+<wire x1="60.96" y1="180.34" x2="60.96" y2="193.04" width="0.1524" layer="91"/>
+<junction x="60.96" y="193.04"/>
 </segment>
 </net>
@@
 <wire x1="76.2" y1="241.3" x2="127" y2="241.3" width="0.1524" layer="91"/>
 <junction x="76.2" y="185.42"/>
-<wire x1="76.2" y1="185.42" x2="25.4" y2="185.42" width="0.1524" layer="91"/>
+<wire x1="76.2" y1="185.42" x2="55.88" y2="185.42" width="0.1524" layer="91"/>
 <label x="30.48" y="185.42" size="1.778" layer="95"/>
 <pinref part="CON3" gate="G$1" pin="2"/>
 <pinref part="CON1" gate="G$1" pin="2"/>
+<wire x1="55.88" y1="185.42" x2="25.4" y2="185.42" width="0.1524" layer="91"/>
 <wire x1="15.24" y1="185.42" x2="25.4" y2="185.42" width="0.1524" layer="91"/>
 <junction x="25.4" y="185.42"/>
@@
 <label x="76.2" y="205.74" size="1.778" layer="95" rot="R90"/>
 <label x="63.5" y="218.44" size="1.778" layer="95"/>
-</segment>
-</net>
+<pinref part="D2" gate="G$1" pin="2"/>
+<wire x1="55.88" y1="180.34" x2="55.88" y2="185.42" width="0.1524" layer="91"/>
+<junction x="55.88" y="185.42"/>
+</segment>
+</net>
