File: PCB/MirZ21_Sub-D.brd (EAGLE design)
At the start: 65.2 x 45.6 mm, 32 parts, among them CON1 M04B4B-ZR4P, CON3 M04, IC1 7805, J1 SOLDERJUMPERTRACE, T1 CON-HARTING-ML_ML4ML4_FEMALE

Commit message: Platine Ver. 2.0
- Korrigierte Märklin Stecker Pins
- CAN Schutzdiode hinzugefügt
- Bohrloch D1 vergrößert
Parts:
- added D2: PESD1CAN, diode:SOT23
- IC1: value 7805 -> 5V
- renumbered U$1 to MOD2, U$2 to MOD1, U$5 to CAN2, U$6 to MOD3
Connections:
- net N$1 renamed CS
- net N$11 renamed RX
- net N$13 renamed LED_TAST
- net N$16 renamed SPK+
- net N$2 renamed SI
- net N$21 renamed MOD2_D18
- net N$22 renamed MOD2_D23
- net N$23 renamed D13
- net N$24 renamed D12
- net N$25 renamed D14
- net N$26 renamed D27
- net N$27 renamed D26
- net N$28 renamed D33
- net N$29 renamed D32
- net N$3 renamed SO_RX
- net N$30 renamed D35
- net N$31 renamed D31
- net N$34 renamed POWER_IN_SV2
- net N$35 renamed POWER_CAN
- net N$4 renamed LED1
- net N$5 renamed CLK
- net N$6 renamed TX
- net N$7 renamed SO
- net N$8 renamed MOD2_D15
- net N$9 renamed EN
- net CAN_H: now also CON1.3, CON3.3, D2.1; no longer CON1.1, CON3.1
- net CAN_L: now also D2.2
- net GND: now also CON1.1, CON3.1, D2.3; no longer CON1.3, CON3.3
Routing:
- net GND: track 247.3 -> 265.0 mm, vias 0 -> 1
- net CAN_H: track 51.9 -> 61.5 mm
- net CAN_L: track 61.4 -> 58.3 mm, vias 1 -> 0
- net SO: track 30.5 -> 32.5 mm
- net SPK+: track 102.2 -> 104.1 mm
- net IR: track 160.0 -> 160.6 mm
Other:
- board text added: "Schwarz"
- board text removed: "Orange"
