File: PCB/MirZ21_Sub-D.sch (EAGLE design)
At the start: 32 parts, among them CON1 M04B4B-ZR4P, CON3 M04, IC1 7805, J1 SOLDERJUMPERTRACE, T1 CON-HARTING-ML_ML4ML4_FEMALE

Commit message: Platine Ver. 2.0
- Korrigierte Märklin Stecker Pins
- CAN Schutzdiode hinzugefügt
- Bohrloch D1 vergrößert
Parts:
- added D2: PESD1CAN, diode:PESD1CAN
- IC1: value 7805 -> 5V
- renumbered U$1 to MOD2, U$2 to MOD1, U$5 to CAN2, U$6 to MOD3
Connections:
- net N$1 renamed CS
- net N$11 renamed RX
- net N$13 renamed LED_TAST
- net N$16 renamed SPK+
- net N$2 renamed SI
- net N$21 renamed MOD2_D18
- net N$22 renamed MOD2_D23
- net N$23 renamed D13
- net N$24 renamed D12
- net N$25 renamed D14
- net N$26 renamed D27
- net N$27 renamed D26
- net N$28 renamed D33
- net N$29 renamed D32
- net N$3 renamed SO_RX
- net N$30 renamed D35
- net N$31 renamed D31
- net N$34 renamed POWER_IN_SV2
- net N$35 renamed POWER_CAN
- net N$4 renamed LED1
- net N$5 renamed CLK
- net N$6 renamed TX
- net N$7 renamed SO
- net N$8 renamed MOD2_D15
- net N$9 renamed EN
- net CAN_H: now also CON1.3, CON3.3, D2.1; no longer CON1.1, CON3.1
- net CAN_L: now also D2.2
- net GND: now also CON1.1, CON3.1, D2.3; no longer CON1.3, CON3.3
Other:
- note added: "02.07.2023"
- note added: "2.0"
- note added: "CAN Kabel von MS2 Märklin E146781 Wrong Pin sequence used in Version 1.0: 1 CAN H Orange 2 CAN L Braun 3 GND Schwarz 4 +18V Rot Black and Orange have to be swapped Correct sequence V 2.0: 1 GND Schwarz 2 CAN L Braun 3 CAN H Orange 4 +18V Rot"
- note added: "CAN2 ohne Fassung bestücken wegen der Höhe . J1 kann zu Tests mit dem CAN Modul getrennt werden und dann mit JP1 überbrückt werden."
- note added: "D4 is only needed if SV2 is used If not D3 could also be bridged."
- note added: "IC1"
- note added: "Revision History: 13.04.22 - Renamed U$ parts - Added names to al nets - Changed drill hole D1 to 0.85mm (Old 0.7mm) 02.07.23:- Corrected Märklin conector pins - Added CAN protection diode D2"
- note added: "ToDo: - ESP32 ein bisschen nach rechts verschieben weil es Versionen gibt welche nicht in das Gehäuse passen Done: - Pinbelegung Märklin Kabel korrigieren - Bohrlöcher für D1 sind zu klein - PESD2CAN platzieren"
- note removed: "13.04.2022"
- note removed: "1a"
- note removed: "CAN Kabel von MS2 Märklin E146781 Wrong Pin sequence used in Version 1.0: CAN H Orange CAN L Braun GND Schwarz +18V Rot Black and Orange have to be swapped Correct sequence: +18V Rot CAN H Orange CAN L Braun GND Schwarz"
- note removed: "U$5 ohne Fassung bestücken wegen der Höhe . J1 kann zu Tests mit dem CAN Modul getrennt werden und dann mit JP1 überbrückt werden."
